File: Hardware/PCB.brd (EAGLE design)
At the start: 46 x 35 mm, 96 parts, among them IC1 BQ25180YBGR, IC2 RV2605YZFR, IC3 BMA423, IC9 RT6160AWSC, J1 503480-2400, J2 TC2030-IDC, J4 KH-TYPE-C-16P, Q1 20V/4.2A/52mΩ/1.4W, Q3 SI1308EDL-T1-GE3, U1 NRF52840_QF, U3 MAX17048G+T10

Commit message: Add files via upload
updated schematic and pcb
Parts:
- removed D1: MBR0530, InkTime_v5:ESP32_C6_LIBRARY_5_SOD3716X135N
- removed R1_EP_DR1: 0.47, InkTime_v5:CPF0201D7K68C1_0201
- added ANT1: 450AT18B100E, InkTime_v5:2450AT18B100E_ANTC3216X140N
- added C1, C17, C18, C2: 12pF, InkTime_v5:NORDIC_NRF_3_RESC0201_L
- added C22: N.C., InkTime_v5:NORDIC_NRF_3_RESC0201_L
- added C4: 1pF, InkTime_v5:NORDIC_NRF_3_RESC0201_L
- added D5: MBR0530, InkTime_v5:ESP32_C6_LIBRARY_5_SOD3716X135N
- added R1_EP_DR: 0.47, InkTime_v5:CPF0201D7K68C1_0201
- added X1: 32MHz, InkTime_v5:NORDIC_NRF_BT-XTAL_2016_N
- added X2: 32.768kHz, Frequency-Source:XTAL330X1051X90N
- L1: value 1.9nH -> 3.9nH; device InkTime_v5:NORDIC_NRF_2_RESC0805_M -> InkTime_v5:NORDIC_NRF_2_RESC0201_M
- L2, L3: device InkTime_v5:NORDIC_NRF_2_RESC0805_M -> InkTime_v5:NORDIC_NRF_2_RESC0402_L
- L5: value 68uH -> 48uH; device InkTime_v5:NORDIC_NRF_2_RESC0805_M -> InkTime_v5:ESP32_C6_LIBRARY_2_IND_4828-WE-TPC_WRE
- moved C3 308.1 mm to (56.3, 140.1)
- moved L1 295.8 mm to (51.2, 122.2)
- moved C11 294.7 mm to (56.1, 135.9)
- moved C7 281.3 mm to (52.5, 140.6)
- moved C8 278.7 mm to (43.2, 138.4)
- moved C10 278.1 mm to (24.4, 132.1)
- moved C21 277.9 mm to (54.2, 141.0)
- moved C20 267.5 mm to (56.1, 137.9)
- moved C9 264.5 mm to (39.4, 117.0)
- moved C5 257.7 mm to (52.5, 134.1)
- moved C12 246.9 mm to (41.8, 142.2)
- moved C13 243.4 mm to (41.9, 143.5)
- moved C6 235.4 mm to (18.0, 122.2)
- moved C16 225.7 mm to (46.2, 119.0)
- moved C15 224.4 mm to (48.5, 120.4)
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Connections:
- removed net BUSY: J1.9
- removed net N$3 (its old number): TP_ON.TP
- removed net SCLI: IC3.12
- new net N$35: C1.2, U1.P$B24, X1.1
- new net N$36: C2.2, U1.P$A23, X1.3
- net 3V3: now also L5.2; no longer L5.1
- net EPD_BUSY: now also J1.9
- net GND: now also C1.1, C17.2, C18.2, C2.1, C22.1, C29.2, C30.2, C31.2, C4.1, IC2.B1, SW_DN.1, SW_ENT.1, SW_UP.1, X1.2, X1.4
- net N$1: now also ANT1.1, C22.2, C4.2, L1.2; no longer IC2.B1
- net N$14: now also D5.2, L5.1; no longer D1.2, L5.2
- net N$18: now also R1_EP_DR.1; no longer R1_EP_DR1.1
- net N$28: now also C17.1, X2.2
- net N$30: now also C18.1, X2.1
- net OUT-: now also TP_ON.TP
- net PREVGH: now also D5.1; no longer D1.1
- net RESE: now also R1_EP_DR.2; no longer R1_EP_DR1.2
- net SCL: now also IC3.12
Routing:
- net GND: track 0.00 -> 386.0 mm, vias 0 -> 12
- net 3V3: track 0.00 -> 199.9 mm, vias 0 -> 24
- net SCL: track 0.00 -> 113.0 mm, vias 0 -> 6
- net SDA: track 0.00 -> 93.7 mm, vias 0 -> 14
- net RESET: track 0.00 -> 85.1 mm, vias 0 -> 8
- net VBUS: track 0.00 -> 84.8 mm, vias 0 -> 9
- net N$26: track 0.00 -> 72.0 mm, vias 0 -> 10
- net N$22: track 0.00 -> 64.4 mm, vias 0 -> 4
- net VBAT: track 0.00 -> 63.4 mm, vias 0 -> 9
- net HAPTIC_EN: track 0.00 -> 61.2 mm
- net P1.01: track 0.00 -> 60.5 mm, vias 0 -> 7
- net RESE: track 0.00 -> 53.2 mm, vias 0 -> 4
- net N$6: track 0.00 -> 50.2 mm, vias 0 -> 5
- net PREVGH: track 0.00 -> 48.1 mm, vias 0 -> 5
- net PREVGL: track 0.00 -> 44.3 mm, vias 0 -> 3
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- added copper zone on layer 1, net GND
- added copper zone on layer 16, net GND
Other:
- outline, holes or cut-outs redrawn
