File: Hardware/Schematic.sch (EAGLE design)
At the start: 96 parts, among them IC1 BQ25180YBGR, IC2 RV2605YZFR, IC3 BMA423, IC9 RT6160AWSC, J1 503480-2400, J2 TC2030-IDC, J4 KH-TYPE-C-16P, Q1 20V/4.2A/52mΩ/1.4W, Q3 SI1308EDL-T1-GE3, U1 NRF52840_QF, U3 MAX17048G+T10

Commit message: Add files via upload
updated schematic and pcb
Parts:
- added ANT1: 450AT18B100E, InkTime_v5:2450AT18B100E_2450AT18B100E
- added C1, C17, C18, C2: 12pF, InkTime_v5:NORDIC_NRF_3_CAPACITOR_0201_L
- added C22: N.C., InkTime_v5:NORDIC_NRF_3_CAPACITOR_0201_L
- added C4: 1pF, InkTime_v5:NORDIC_NRF_3_CAPACITOR_0201_L
- added X1: 32MHz, InkTime_v5:NORDIC_NRF_XTAL_32MHZ
- added X2: 32.768kHz, Frequency-Source:9HT10
- L1: value 1.9nH -> 3.9nH; device InkTime_v5:NORDIC_NRF_2_INDUCTOR_0805_M -> InkTime_v5:NORDIC_NRF_2_INDUCTOR_0201_M
- L2, L3: device InkTime_v5:NORDIC_NRF_2_INDUCTOR_0805_M -> InkTime_v5:NORDIC_NRF_2_INDUCTOR_0402_L
- L5: value 68uH -> 48uH; device InkTime_v5:NORDIC_NRF_2_INDUCTOR_0805_M -> InkTime_v5:ESP32_C6_LIBRARY_2_744043680IND_4828-WE-TPC_WRE
- renumbered D1 to D5, R1_EP_DR1 to R1_EP_DR
Connections:
- removed net BUSY: J1.9
- removed net N$3 (its old number): TP_ON.TP
- removed net SCLI: IC3.SCX
- new net N$35: C1.2, U1.XC1@B24, X1.1
- new net N$36: C2.2, U1.XC2@A23, X1.3
- net 3V3: now also L5.2; no longer L5.1
- net EPD_BUSY: now also J1.9
- net GND: now also C1.1, C17.2, C18.2, C2.1, C22.1, C29.2, C30.2, C31.2, C4.1, IC2.IN/TRIG, SW_DN.1, SW_ENT.1, SW_UP.1, X1.2, X1.4
- net N$1: now also ANT1.FEED, C22.2, C4.2, L1.2; no longer IC2.IN/TRIG
- net N$14: now also L5.1; no longer L5.2
- net N$28: now also C17.1, X2.2
- net N$30: now also C18.1, X2.1
- net OUT-: now also TP_ON.TP
- net SCL: now also IC3.SCX
Other:
- note added: "DEC1"
- moved on the sheet: SW_DN, SW_ENT, SW_UP, TP_3.3V, TP_GND, TP_RESET, TP_SWDIO, TP_SWD_CLK, TP_SWO
